File: hardware/addon-keys/addon-keys.kicad_pcb (KiCad board)
At the start: 2 copper layers, 83.4 x 79.9 mm, 28 parts, among them J1 GUITION H1, J2 5V IN (+ -), J3 USB-C 5V (optional), J4 SWIO 3V3 GND, SW1 KEY 1, SW2 KEY 2, SW3 KEY 3, U1 LDL1117S33R, U2 CH32V003A4M6, U3 HLK-LD2402, U5 SHT40-AD1B-R2

Commit message: Centre the radar under key 2, add spare pads and test points
Keys board: the radar break-away piece is now centred under key 2,
0.3 mm below its switch body (as close as it can go). It has 1 mm gaps
down each side and three bridges: the traces bridge in the left side
gap, one in the top gap right of key 2's socket, one in the right side
gap.

Both boards: J5 brings the panel's IO40 and UART0 and the CH32V003's
PA2 and PD7 (NRST) out to 2.54 mm pads with GND, and TP1-TP8 put test
points on 5V, 3V3, GND, SDA, SCL and the radar's TX, RX and OUT. The
alignment STL widens J5's holes like the other headers.

Co-Authored-By: Claude Opus 5.5 <noreply@anthropic.com>
Parts:
- added J5: SPARE, Connector_PinHeader_2.54mm:PinHeader_1x06_P2.54mm_Vertical, B.Cu at (112.0, 139.4)
- added TP1: +5V, TestPoint:TestPoint_Pad_D1.5mm, B.Cu at (128.5, 139.4)
- added TP2: +3V3, TestPoint:TestPoint_Pad_D1.5mm, B.Cu at (131.5, 139.4)
- added TP3: GND, TestPoint:TestPoint_Pad_D1.5mm, B.Cu at (134.5, 139.4)
- added TP4: SDA, TestPoint:TestPoint_Pad_D1.5mm, B.Cu at (137.5, 139.4)
- added TP5: SCL, TestPoint:TestPoint_Pad_D1.5mm, B.Cu at (140.5, 139.4)
- added TP6: RADAR_TX, TestPoint:TestPoint_Pad_D1.5mm, B.Cu at (143.5, 139.4)
- added TP7: RADAR_RX, TestPoint:TestPoint_Pad_D1.5mm, B.Cu at (146.5, 139.4)
- added TP8: RADAR_OUT, TestPoint:TestPoint_Pad_D1.5mm, B.Cu at (149.5, 139.4)
- moved MB2 31.4 mm to (150.4, 161.6)
- moved MB3 31.4 mm to (155.2, 165.0)
- moved U3 31.4 mm to (143.7, 169.9)
- moved MB1 26.9 mm to (132.2, 165.0), turned to 90 degrees
Connections:
- J1 pad 3: unconnected-(J1-Pin_3-Pad3) -> /IO40
- J1 pad 4: unconnected-(J1-Pin_4-Pad4) -> /U0RXD
- J1 pad 6: unconnected-(J1-Pin_6-Pad6) -> /U0TXD
- U2 pad 11: unconnected-(U2-PD7-Pad11) -> /PD7
- U2 pad 13: unconnected-(U2-PA2-Pad13) -> /PA2
Other:
- outline, holes or cut-outs redrawn
- board text added: "3V3"
- board text added: "5V"
- board text added: "IO40"
- board text added: "PA2"
- board text added: "PD7"
- board text added: "R-OUT"
- board text added: "R-RX"
- board text added: "R-TX"
- board text added: "RXD"
- board text added: "SCL"
- board text added: "SDA"
- board text added: "TXD"
