File: hardware/addon-keys/addon-keys.kicad_sch (KiCad schematic)
At the start: 25 parts, among them J1 GUITION H1, J2 5V IN (+ -), J3 USB-C 5V (optional), J4 SWIO 3V3 GND, SW1 KEY 1, SW2 KEY 2, SW3 KEY 3, U1 LDL1117S33R, U2 CH32V003A4M6, U3 HLK-LD2402, U5 SHT40-AD1B-R2

Commit message: Centre the radar under key 2, add spare pads and test points
Keys board: the radar break-away piece is now centred under key 2,
0.3 mm below its switch body (as close as it can go). It has 1 mm gaps
down each side and three bridges: the traces bridge in the left side
gap, one in the top gap right of key 2's socket, one in the right side
gap.

Both boards: J5 brings the panel's IO40 and UART0 and the CH32V003's
PA2 and PD7 (NRST) out to 2.54 mm pads with GND, and TP1-TP8 put test
points on 5V, 3V3, GND, SDA, SCL and the radar's TX, RX and OUT. The
alignment STL widens J5's holes like the other headers.

Co-Authored-By: Claude Opus 5.5 <noreply@anthropic.com>
Parts:
- added J5: SPARE, Connector_PinHeader_2.54mm:PinHeader_1x06_P2.54mm_Vertical, symbol Connector_Generic:Conn_01x06
- added TP1: +5V, TestPoint:TestPoint_Pad_D1.5mm, symbol Connector:TestPoint
- added TP2: +3V3, TestPoint:TestPoint_Pad_D1.5mm, symbol Connector:TestPoint
- added TP3: GND, TestPoint:TestPoint_Pad_D1.5mm, symbol Connector:TestPoint
- added TP4: SDA, TestPoint:TestPoint_Pad_D1.5mm, symbol Connector:TestPoint
- added TP5: SCL, TestPoint:TestPoint_Pad_D1.5mm, symbol Connector:TestPoint
- added TP6: RADAR_TX, TestPoint:TestPoint_Pad_D1.5mm, symbol Connector:TestPoint
- added TP7: RADAR_RX, TestPoint:TestPoint_Pad_D1.5mm, symbol Connector:TestPoint
- added TP8: RADAR_OUT, TestPoint:TestPoint_Pad_D1.5mm, symbol Connector:TestPoint
- J1: Note plugs into the panel's H1; SDA = IO1 (pin 7), SCL = IO2 (pin 5); IO40 and the ESP's UART0 (pins 4, 6) unused. Needs R25-R27 fitted on the panel. -> plugs into the panel's H1; SDA = IO1 (pin 7), SCL = IO2 (pin 5); IO40 and the ESP's UART0 (pins 3, 4, 6) go to the spare pads J5. Needs R25-R27 fitted on the panel.
- U2: Note PD5 = USART1 TX, PD6 = RX; PC1/PC2 = I2C1; PD7 (NRST) and PA2 spare -> PD5 = USART1 TX, PD6 = RX; PC1/PC2 = I2C1; PD7 (NRST) and PA2 spare, on J5
Connections:
- net +3V3: now also TP2.1
- net +5V: now also TP1.1
- net GND: now also J5.6 (Pin_6), TP3.1
- net RADAR_OUT: now also TP8.1
- net RADAR_RX: now also TP7.1
- net RADAR_TX: now also TP6.1
- net SCL: now also TP5.1
- net SDA: now also TP4.1
- net IO40: now reaches J1.3 (Pin_3)
- net IO40: now also J5.1 (Pin_1)
- net U0RXD: now reaches J1.4 (Pin_4)
- net U0RXD: now also J5.2 (Pin_2)
- net U0TXD: now reaches J1.6 (Pin_6)
- net U0TXD: now also J5.3 (Pin_3)
- net PD7: now reaches U2.11 (PD7)
- net PD7: now also J5.5 (Pin_5)
- net PA2: now reaches U2.13 (PA2)
- net PA2: now also J5.4 (Pin_4)
- no-connect marks 5 -> 0
Other:
- note added: "Radar: HLK-LD2402 soldered on its own 2.5 mm header, antenna side out, on a break-away piece centred under key 2 (snap it off to build without the radar). Check the module's print: 1 VCC, 2 OUT, 3 GND, 4 TX, 5 RX (Hi-Link manual p. 7)."
- note added: "Spare pins on J5 (2.54 mm pads for wires): the panel's IO40 and UART0 from H1, the co-processor's PA2 and PD7 (NRST), and GND. Test points TP1-TP8 (1.5 mm pads on the back): 5 V, 3.3 V, GND, I2C and the radar's UART and OUT."
- note removed: "Radar: HLK-LD2402 soldered on its own 2.5 mm header, antenna side out, on a break-away piece at the bar's left end, under key 1 (snap it off to build without the radar). Check the module's print: 1 VCC, 2 OUT, 3 GND, 4 TX, 5 RX (Hi-Link manual p. 7)."
